Commit message: Include all collision geometry in relevant Franka URDF; achieve proper coordinate frame for end effector tip

File: assets/franka_with_ee_full_collisions.urdf (robot description, URDF)
Before this commit: robot panda, 11 links, 10 joints
Links:
- link end_effector_link: geometry collision cylinder length=0.1016 radius=0.0127; visual cylinder length=0.1016 radius=0.0127
Joints:
- joint fix_tip_link: origin xyz=0 0 -0.1169 rpy=0 0 0 -> xyz=0 0 -0.1169 rpy=3.141592654 0 0
